File: CalibratedPhotoDiodeTriax/CalibratedPhotoDiodeTriax.kicad_sch (KiCad schematic)
At the start: 2 parts, among them J1 TO-5 Photodiode Socket: Conn_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, J2 CBJ70 Triax Throughhole Conne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

Commit message: Trying to revise accessibility
Connections:
- net GND: now also J1.2 (Pin_2); no longer J1.3 (Pin_3)
- net at J2.2 (In2): now also J1.3 (Pin_3); no longer J1.2 (Pin_2)
Changed lines of the file:
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@@
 	(paper "A4")
 	(junction
-		(at 157.48 60.96)
+		(at 154.94 62.23)
 		(diameter 0)
 		(color 0 0 0 0)
@@
 	(wire
 		(pts
-			(xy 154.94 63.5) (xy 154.94 59.69)
-		)
-		(stroke
-			(width 0)
-			(type default)
-		)
-	)
-	(wire
-		(pts
-			(xy 157.48 66.04) (xy 157.48 60.96)
-		)
-		(stroke
-			(width 0)
-			(type default)
-		)
-	)
-	(wire
-		(pts
-			(xy 160.02 71.12) (xy 160.02 63.5)
-		)
-		(stroke
-			(width 0)
-			(type default)
-		)
-	)
-	(wire
-		(pts
 			(xy 149.86 59.69) (xy 152.4 59.69)
 		)
@@
 	(wire
 		(pts
-			(xy 160.02 63.5) (xy 154.94 63.5)
-		)
-		(stroke
-			(width 0)
-			(type default)
-		)
-	)
-	(wire
-		(pts
-			(xy 157.48 60.96) (xy 157.48 59.69)
-		)
-		(stroke
-			(width 0)
-			(type default)
-		)
-	)
-	(wire
-		(pts
-			(xy 154.94 66.04) (xy 157.48 66.04)
-		)
-		(stroke
-			(width 0)
-			(type default)
-		)
-	)
-	(wire
-		(pts
-			(xy 157.48 60.96) (xy 162.56 60.96)
+			(xy 157.48 59.69) (xy 157.48 64.77)
+		)
+		(stroke
+			(width 0)
+			(type default)
+		)
+	)
+	(wire
+		(pts
+			(xy 154.94 59.69) (xy 154.94 62.23)
+		)
+		(stroke
+			(width 0)
+			(type default)
+		)
+	)
+	(wire
+		(pts
+			(xy 157.48 64.77) (xy 160.02 64.77)
+		)
+		(stroke
+			(width 0)
+			(type default)
+		)
+	)
+	(wire
+		(pts
+			(xy 154.94 62.23) (xy 163.83 62.23)
+		)
+		(stroke
+			(width 0)
+			(type default)
+		)
+	)
+	(wire
+		(pts
+			(xy 154.94 62.23) (xy 154.94 66.04)
+		)
+		(stroke
+			(width 0)
+			(type default)
+		)
+	)
+	(wire
+		(pts
+			(xy 160.02 64.77) (xy 160.02 71.12)
 		)
 		(stroke
@@
 	(symbol
 		(lib_id "power:GND")
-		(at 162.56 60.96 0)
+		(at 163.83 62.23 0)
 		(unit 1)
 		(exclude_from_sim no)
@@
 		(fields_autoplaced yes)
 		(property "Reference" "#PWR01"
-			(at 162.56 67.31 0)
+			(at 163.83 68.58 0)
 			(effects
 				(font
@@
 		)
 		(property "Value" "GND"
-			(at 162.56 66.04 0)
+			(at 163.83 67.31 0)
 			(effects
 				(font
@@
 		)
 		(property "Footprint" ""
-			(at 162.56 60.96 0)
+			(at 163.83 62.23 0)
 			(effects
 				(font
@@
 		)
 		(property "Datasheet" ""
-			(at 162.56 60.96 0)
+			(at 163.83 62.23 0)
 			(effects
 				(font
@@
 		)
 		(property "Description" "Power symbol creates a global label with name \"GND\" , ground"
-			(at 162.56 60.96 0)
-			(effects
-				(font
+			(at 163.83 62.23 0)
+			(effects
+				(font
